Commit message: Lastest update: Still facing errors when using rviz with map server

File: src/ansrrbot/xacro/ansrr_bot.xacro (robot description, xacro)
@@ -1,4 +1,4 @@
 <?xml version="1.0" encoding="UTF-8"?>
-<robot xmlns:xacro="http://www.ros.org/wiki/xacro" name="ansrr">
+<robot xmlns:xacro="http://www.ros.org/wiki/xacro" name="ansrr_bot">
   <xacro:include filename="$(cwd)/macs.xacro" />
   <link name="base_link">
@@ -39,6 +39,14 @@
   <gazebo>
     <plugin name="differential_drive_controller" filename="libgazebo_ros_diff_drive.so">
-      <leftJoint>[base_to_left_rear,base_to_left_front]</leftJoint>
-      <rightJoint>[base_to_right_rear,base_to_right_front]</rightJoint>
+      <leftJoint>base_to_left_rear</leftJoint>
+      <rightJoint>base_to_right_rear</rightJoint>
+      <robotBaseFrame>base_link</robotBaseFrame>
+      <wheelSeparation>0.4064</wheelSeparation>
+      <wheelDiameter>${wheel_radius*2}</wheelDiameter>
+      <publishWheelJointState>true</publishWheelJointState>
+    </plugin>
+    <plugin name="differential_drive_controller" filename="libgazebo_ros_diff_drive.so">
+      <leftJoint>base_to_left_front</leftJoint>
+      <rightJoint>base_to_right_front</rightJoint>
       <robotBaseFrame>base_link</robotBaseFrame>
       <wheelSeparation>0.4064</wheelSeparation>
@@ -68,5 +76,5 @@
       </ray>
       <plugin name="gazebo_ros_lds_lfcd_controller  " filename="libgazebo_ros_laser.so">
-        <topicName>/raw_scan</topicName>
+        <topicName>/scan</topicName>
         <frameName>lidar</frameName>
       </plugin>

File: src/ansrrbot/xacro/macs.xacro (robot description, xacro)
@@ -112,4 +112,10 @@
     <origin rpy="1.5708 0 0" xyz="${x} ${y} ${z}"/>
   </joint>
+  <transmission name="${w_name}_joint_trans" type="SimpleTransmission">
+      <actuator name="${w_name}_motor"/>
+      <joint name="$base_to_{w_name}"/>
+      <mechanicalReduction>1</mechanicalReduction>
+      <motorTorqueConstant>1</motorTorqueConstant>
+  </transmission>
 </xacro:macro>
 </robot>
