Commit message: Fixed Orientation of the wheels to rectify incorrect move_base action

File: src/ansrrbot/xacro/ansrr_bot.urdf (robot description, URDF)
Before this commit: robot ansrr_bot, 11 links, 10 joints
Joints:
- joint base_to_left_front: origin xyz=-0.1524 -0.25 -0.06096 rpy=1.5708 0 0 -> xyz=0.1524 0.25 -0.06096 rpy=1.5708 0 3.14
- joint base_to_left_rear: origin xyz=0.1524 -0.25 -0.06096 rpy=1.5708 0 0 -> xyz=-0.1524 0.25 -0.06096 rpy=1.5708 0 3.14
- joint base_to_lidar: origin xyz=-.2286 0 0.1 rpy=0 0 3.14 -> xyz=-.2286 0 0.1 rpy=0 0 0
- joint base_to_right_front: origin xyz=-0.1524 0.25 -0.06096 rpy=1.5708 0 0 -> xyz=0.1524 -0.25 -0.06096 rpy=1.5708 0 3.14
- joint base_to_right_rear: origin xyz=0.1524 0.25 -0.06096 rpy=1.5708 0 0 -> xyz=-0.1524 -0.25 -0.06096 rpy=1.5708 0 3.14

File: src/ansrrbot/xacro/ansrr_bot.xacro (robot description, xacro)
@@ -14,8 +14,8 @@
     <xacro:inertia_macro mass="1" ixx= "${box_ixx}" iyy="${box_iyy}" izz="${box_izz}"/>
   </link>
-  <xacro:wheel w_name="left_front" x="${front_x}" y="-${wheel_y}" z="${wheel_z}"/>
-  <xacro:wheel w_name="left_rear" x="${rear_x}" y="-${wheel_y}" z="${wheel_z}"/>
-  <xacro:wheel w_name="right_front" x="${front_x}" y="${wheel_y}" z="${wheel_z}"/>
-  <xacro:wheel w_name="right_rear" x="${rear_x}" y="${wheel_y}" z="${wheel_z}"/>
+  <xacro:wheel w_name="left_front" x="${front_x}" y="${wheel_y}" z="${wheel_z}"/>
+  <xacro:wheel w_name="left_rear" x="${rear_x}" y="${wheel_y}" z="${wheel_z}"/>
+  <xacro:wheel w_name="right_front" x="${front_x}" y="-${wheel_y}" z="${wheel_z}"/>
+  <xacro:wheel w_name="right_rear" x="${rear_x}" y="-${wheel_y}" z="${wheel_z}"/>
   <link name="lidar">
     <visual>
@@ -35,5 +35,5 @@
     <parent link="base_link"/>
     <child link="lidar"/>
-    <origin rpy="0 0 3.14" xyz="-.2286 0 0.1"/>
+    <origin rpy="0 0 0" xyz="-.2286 0 0.1"/>
   </joint>
   <gazebo>

File: src/ansrrbot/xacro/macs.xacro (robot description, xacro)
@@ -14,6 +14,6 @@
 <xacro:property name="wheel_iyy" value= "5.685e-4"/>
 <xacro:property name="wheel_izz" value= "2.903e-4"/>
-<xacro:property name="front_x" value="-0.1524"/>
-<xacro:property name="rear_x" value="0.1524"/>
+<xacro:property name="front_x" value="0.1524"/>
+<xacro:property name="rear_x" value="-0.1524"/>
 <xacro:property name="wheel_y" value="0.25"/>
 <xacro:property name="wheel_z" value="-0.06096"/>
@@ -110,5 +110,5 @@
     <parent link="base_link"/>
     <child link="${w_name}"/>
-    <origin rpy="1.5708 0 0" xyz="${x} ${y} ${z}"/>
+    <origin rpy="1.5708 0 3.14" xyz="${x} ${y} ${z}"/>
   </joint>
   <transmission name="${w_name}_joint_trans" type="SimpleTransmission">
