Commit message: Added Elec Box to Ansrr_v2. Updated Inertial parameters of the xacro file.

File: src/ansrrbot/xacro/ansrr_v2.xacro (robot description, xacro)
@@ -52,4 +52,28 @@
             xyz="${wheel_right['pos_x']} ${wheel_right['pos_y']} ${wheel_right['pos_z']}"/>
   </joint>
+  <link name="elec_box">
+    <visual>
+      <geometry>
+        <box size="${elec_box['x']} ${elec_box['y']} ${elec_box['z']}"/>
+      </geometry>
+      <material name="aluminium_silver"/>
+    </visual>
+    <collision>
+      <geometry>
+        <box size="${elec_box['x']} ${elec_box['y']} ${elec_box['z']}"/>
+      </geometry>
+    </collision>
+    <inertial>
+      <mass value="${elec_box['mass']}"/>
+      <inertia ixx="${elec_box['ixx']}" ixy="0" ixz="0" iyy="${elec_box['iyy']}" iyz="0" izz="${elec_box['izz']}"/>
+    </inertial>
+  </link>
+  <joint name="base_to_elec_box" type="fixed">
+    <axis xyz="0 0 1"/>
+    <parent link="base_link"/>
+    <child link="elec_box"/>
+    <origin rpy="${elec_box_ref['rot_r']} ${elec_box_ref['rot_p']} ${elec_box_ref['rot_y']}"
+            xyz="${elec_box_ref['pos_x']} ${elec_box_ref['pos_y']} ${elec_box_ref['pos_z']}"/>
+  </joint>
   <gazebo>
     <plugin filename="libgazebo_ros_diff_drive.so" name="differential_drive_controller">

File: src/ansrrbot/xacro/macs_v2.xacro (robot description, xacro)
@@ -11,4 +11,6 @@
   <xacro:property name="motor_right" value="${params['motor_right']}" />
   <xacro:property name="base_link" value="${params['base_link']}" />
+  <xacro:property name="elec_box" value="${params['elec_box']}" />
+  <xacro:property name="elec_box_ref" value="${params['elec_box_ref']}" />
   <!-- Materials -->
   <material name="tire_black">

Commit message: Updated Xacro

File: src/ansrrbot/xacro/ansrr_v2.xacro (robot description, xacro)
@@ -52,4 +52,5 @@
             xyz="${wheel_right['pos_x']} ${wheel_right['pos_y']} ${wheel_right['pos_z']}"/>
   </joint>
+  <link name="elec_box">
   <gazebo>
     <plugin filename="libgazebo_ros_diff_drive.so" name="differential_drive_controller">
