Commit message: Last Update on Project used for Presenation

File: src/ansrrbot/urdf/urdf_v3.urdf (robot description, URDF)
Before this commit: robot ansrrbot, 22 links, 21 joints
Joints:
- joint jnt_base_frame_to_lidar: origin xyz=-0.178 -0.155 0.000199999999999367 rpy=1.57079632679 0 0 -> xyz=-0.178 -0.155 0 rpy=1.5707 0 0
